Commit message: update ros2_control params for new waveshare_servos, use joint_state_publisher_gui

File: urdf/lekiwi.ros2_control.xacro (robot description, xacro)
@@ -5,6 +5,6 @@
     <hardware>
       <plugin>waveshare_servos/WaveshareServos</plugin>
-      <param name="usb_port">/dev/ttyACM0</param>
-      <param name="baud_rate">1000000</param>
+      <param name="port">/dev/ttyACM0</param>
+      <param name="baudrate">1000000</param>
     </hardware>
     <!-- Left wheel servo (ID: 7) -->
@@ -12,11 +12,12 @@
       <param name="id">7</param>
       <param name="type">vel</param>
+      <param name="max_speed">9.2</param>
       <command_interface name="velocity">
-        <param name="min">-10.0</param>
-        <param name="max">10.0</param>
+        <param name="min">-9.2</param>
+        <param name="max">9.2</param>
       </command_interface>
       <state_interface name="position"/>
       <state_interface name="velocity"/>
-      <state_interface name="torque"/>
+      <state_interface name="effort"/>
       <state_interface name="temperature"/>
     </joint>
@@ -25,11 +26,12 @@
       <param name="id">8</param>
       <param name="type">vel</param>
+      <param name="max_speed">9.2</param>
       <command_interface name="velocity">
-        <param name="min">-10.0</param>
-        <param name="max">10.0</param>
+        <param name="min">-9.2</param>
+        <param name="max">9.2</param>
       </command_interface>
       <state_interface name="position"/>
       <state_interface name="velocity"/>
-      <state_interface name="torque"/>
+      <state_interface name="effort"/>
       <state_interface name="temperature"/>
     </joint>
@@ -38,11 +40,12 @@
       <param name="id">9</param>
       <param name="type">vel</param>
+      <param name="max_speed">9.2</param>
       <command_interface name="velocity">
-        <param name="min">-10.0</param>
-        <param name="max">10.0</param>
+        <param name="min">-9.2</param>
+        <param name="max">9.2</param>
       </command_interface>
       <state_interface name="position"/>
       <state_interface name="velocity"/>
-      <state_interface name="torque"/>
+      <state_interface name="effort"/>
       <state_interface name="temperature"/>
     </joint>

File: urdf/omni_base.xacro (robot description, xacro)
@@ -92,8 +92,8 @@
         </geometry>
       </collision>
-      <inertial>
+      <!--<inertial>
         <origin xyz="0 0.003 0" rpy="${-PI/2} 0 0"/>
         <mass value="0.154"/>
-      </inertial>
+      </inertial>-->
     </link>
     <joint name="${prefix}_wheel_joint" type="continuous">
